File: Electronics/KiCAD/APG_Sensor_Test_Board/IMU.kicad_sch (KiCad schematic)
At the start: 9 parts, among them U2 BNO085

Commit message: Edit PCB and Update component values
Parts:
- C5: value 0.1uF -> 1uf
Changed lines of the file:
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@@
 		(lib_id "Device:C_Small")
 		(at 134.62 44.45 0)
-		(mirror y)
 		(unit 1)
 		(exclude_from_sim no)
@@
 		(on_board yes)
 		(dnp no)
-		(fields_autoplaced yes)
 		(property "Reference" "C5"
 			(at 132.08 43.1862 0)
@@
 					(size 1.27 1.27)
 				)
-				(justify left)
+				(justify right)
 			)
 		)
-		(property "Value" "0.1uF"
+		(property "Value" "1uf"
 			(at 132.08 45.7262 0)
 			(effects
@@
 					(size 1.27 1.27)
 				)
-				(justify left)
+				(justify right)
 			)
 		)

Commit message: APG Sensor Board V1.1 Production
Parts:
- C5: value 1uf -> 1uF
Changed lines of the file:
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@@
 			)
 		)
-		(property "Value" "1uf"
+		(property "Value" "1uF"
 			(at 132.08 45.7262 0)
 			(effects
