File: Electronics/KiCAD/APG_Sensor_Test_Board/Power_and_USB.kicad_sch (KiCad schematic)
At the start: 12 parts, among them J4 USB_C_Receptacle_USB2.0_16P, U6 TLV1117-33

Commit message: Layout and routing
Parts:
- removed U6: TLV1117-33, Package_TO_SOT_SMD:SOT-223-3_TabPin2, symbol Regulator_Linear:TLV1117-33
- added D4: SS12, Diode_SMD:D_SMA, symbol Device:D_Schottky
- added U7: TLV75533PDBV, Package_TO_SOT_SMD:SOT-23-5, symbol Regulator_Linear:TLV75533PDBV
- C14: renamed from C17; footprint Capacitor_SMD:C_0805_2012Metric -> Capacitor_SMD:C_0603_1608Metric
- C15: renamed from C14; footprint Capacitor_SMD:C_0805_2012Metric -> Capacitor_SMD:C_0603_1608Metric
- C16: renamed from C15; footprint Capacitor_SMD:C_0805_2012Metric -> Capacitor_SMD:C_0603_1608Metric
- C17: renamed from C16; footprint Capacitor_SMD:C_0805_2012Metric -> Capacitor_SMD:C_0603_1608Metric
- R27, R28: footprint Resistor_SMD:R_0805_2012Metric -> Resistor_SMD:R_0603_1608Metric
- TP20, TP21: footprint TestPoint:TestPoint_Pad_3.0x3.0mm -> TestPoint:TestPoint_Pad_D1.0mm
- U6: renamed from U7; value ~ -> TPCM1293A-04SO; footprint (none) -> Package_TO_SOT_SMD:SOT-23-6; JLCPCB (none) -> C558415
Connections:
- net +3V3: now also U7.5 (OUT)
- net +5V: now also D4.2 (A); no longer C16.1
- net D_N: now also U6.3 (CH2); no longer U6.6 (CH4)
- net D_P: now also U6.1 (CH1); no longer U6.4 (CH3)
- new net: C16.1, D4.1 (K), U7.1 (IN), U7.3 (EN)
Other:
- moved on the sheet: C17, TP21

Commit message: layout changes
Connections:
- net GND: now also U7.2 (GND)
Changed lines of the file:
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@@
+	(wire
+		(pts
+			(xy 203.2 83.82) (xy 203.2 85.09)
+		)
+		(stroke
+			(width 0)
+			(type default)
+		)
+	)
 	(wire
 		(pts
@@
 					(unit 1)
 				)
+			)
+		)
+	)
+	(symbol
+		(lib_id "power:GND")
+		(at 203.2 85.09 0)
+		(unit 1)
+		(exclude_from_sim no)
+		(in_bom yes)
+		(on_board yes)
+		(dnp no)
+		(fields_autoplaced yes)
+		(property "Reference" "#PWR055"
+			(at 203.2 91.44 0)
+			(effects
+				(font
+					(size 1.27 1.27)
+				)
+				(hide yes)
+			)
+		)
+		(property "Value" "GND"
+			(at 203.2 90.17 0)
+			(effects
+				(font
+					(size 1.27 1.27)
+				)
+			)
+		)
+		(property "Footprint" ""
+			(at 203.2 85.09 0)
+			(effects
+				(font
+					(size 1.27 1.27)
+				)
+				(hide yes)
+			)
+		)
+		(property "Datasheet" ""
+			(at 203.2 85.09 0)
+			(effects
+				(font
+					(size 1.27 1.27)
+				)
+				(hide yes)
+			)
+		)
+		(property "Description" "Power symbol creates a global label with name \"GND\" , ground"
+			(at 203.2 85.09 0)
+			(effects
+				(font
+					(size 1.27 1.27)
+				)
+				(hide yes)
+			)
+		)
+		(pin "1"
+		)
+		(instances
+			(project "APG_Sensor_Test_Board"
+				(path "/3161be0c-372f-463d-be0a-bab00f344057/ce24b18a-13e5-44eb-9a8e-7d29741d4106"
+					(reference "#PWR055")
+					(unit 1)
+				)

Commit message: new tvs diode debug changes
Parts:
- removed U6: TPCM1293A-04SO, Package_TO_SOT_SMD:SOT-23-6, symbol Project:CM1293A-04SO
- added U6: USBULC6-2M6, Package_DFN_QFN:ST_UQFN-6L_1.5x1.7mm_P0.5mm, symbol Project:USBULC6-2M6
- C14: value 1u -> 0.1uF
Connections:
- net +5V: no longer C14.1
- net D_N: now also U6.1 (I/O1), U6.6 (I/O1)
- net D_P: now also U6.3 (I/O2), U6.4 (I/O2)
- net GND: now also C14.1, U6.2 (GND); no longer C14.2
- new net: C14.2, U6.5 (CAP)
- no-connect marks 4 -> 2

Commit message: APG Sensor Board V1.1 Production
Parts:
- C16, C17: value 1u -> 1uF
- FB1: value 330Ω -> 330; JLCPCB (none) -> C76819
Changed lines of the file:
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@@
 			)
 		)
-		(property "Value" "1u"
+		(property "Value" "1uF"
 			(at 231.14 78.7462 0)
 			(effects
@@
 			)
 		)
-		(property "Value" "1u"
+		(property "Value" "1uF"
 			(at 179.07 78.7462 0)
 			(effects
@@
 			)
 		)
-		(property "Value" "330Ω"
+		(property "Value" "330"
 			(at 120.5992 77.47 90)
 			(effects
@@
 			(at 120.65 82.55 0)
 			(effects
+				(font
+					(size 1.27 1.27)
+				)
+				(hide yes)
+			)
+		)
+		(property "JLCPCB" "C76819"
+			(at 120.65 82.55 0)
+			(effects
